File: OpenServoDrive.brd (EAGLE design)
At the start: 108.6 x 87 mm, 175 parts, among them IC1 LTC6103, IC11 LMV7219M7, IC12 MCP2515, IC13 HCTL-2032-SC, IC14 74AHCT1G86GW, IC15 MCP2551, IC16 HIP4081A, IC2 HIP4081A, IC3 LD1117S50, IC4 MC34063, IC5 OPA336NJ, IC6 OPA2336UA, IC7 OPA2336UA, IC8 ATMEGA2560-16AU, IC9 LTC6103, J1 Motor 1, J13 Motor 2, J2 60V Motor Power, J3 Regulator Bypass, J4 AREF, J5 Terminator, J7 CAN, J8 Ground, J9 ISP, Q1 AOT414, Q10 AOT414, Q11 16 MHz, Q12 2N7002, Q13 16 MHz, Q2 AOT414, Q3 AOT414, Q4 AOT414, Q5 16 MHz, Q6 2N7002, Q7 AOT414, Q8 AOT414, Q9 AOT414

Commit message: foo
Parts:
- removed C21, C22, C44, C45, C46: 100 nF, rcl:C0805K
- removed C36: 22 pF, rcl:C0805K
- removed C37: 100nF, rcl:C0805K
- removed D2: UF4002, diode:D-7.5
- removed IC4: MC34063, SparkFun:SO08
- removed IC8: ATMEGA2560-16AU, atmel-2005:TQFP100
- removed J8: Ground, jumper:SJ
- removed L1: 220 uH, wuerth-elektronik:WE-PD_L/XL/XXL
- removed LED4: Status, freetronics:LED-0805-LARGE
- removed Q5: 16 MHz, SparkFun:HC49US
- removed R28, R49: 1 k, rcl:M0805
- removed R53: 10 k, rcl:M0805
- removed U$3, U$6, U$7: OSHW-LOGOS, SparkFun:OSHW-LOGO-S
- added C42: 22pF, freetronics-master-v1:0603
- added C43, C54: 100nF, freetronics-master-v1:0603
- added C53, C59: 2.2nF, freetronics-master-v1:0603
- added C55: 10nF, freetronics-master-v1:0603
- added C57: 10µF, freetronics-jon:C1206K
- added C58: 22µF, freetronics-jon:C1206K
- added D18: SK34A-LTP, freetronics-luke:SMA
- added IC10: EUP3476, freetronics-luke:SO08T
- added IC20: ATmega1281, SparkFun:TQFP64_14X14MM
- added L4: 6.8 uH, freetronics-luke:CDRH
- added LED7: 60V, freetronics-master-v1:LED-0603
- added R62: 15k, freetronics-master-v1:0603
- added R63: 53.6k, freetronics-master-v1:0603
- added R64: 10k 1%, freetronics-master-v1:0603
- added R66: 100k, freetronics-master-v1:0603
- added U$55, U$56, U$68: OSHW-LOGOS, SparkFun:OSHW-LOGO-S
- added ZD1: 12.6V, freetronics-luke:MINIMELF
- C11, C15, C39: value 22 pF -> 100nF; device rcl:C0805K -> freetronics-master-v1:0603
- C12, C13: value 100 nF -> 100nF; device rcl:C0805K -> freetronics-master-v1:0603
- C14: value 100 nF -> 22pF; device rcl:C0805K -> freetronics-master-v1:0603
- C16: value 100 nF -> 10nF; device rcl:C0805K -> freetronics-master-v1:0603
- C25, C26, C28: value 10 nF -> 10nF; device rcl:C0805K -> freetronics-master-v1:0603
- C29: value 10 nF -> 100nF; device rcl:C0805K -> freetronics-master-v1:0603
- C38: value 22 pF -> 22pF; device rcl:C0805K -> freetronics-master-v1:0603
- C6: value 100 uF -> 47µF; device resistor:E2,5-6 -> freetronics-jon:C1210
- C7: value 470 pF -> 100nF; device rcl:C0805K -> freetronics-master-v1:0603
- C8: value 470 uF -> 100nF; device resistor:E3,5-8 -> freetronics-master-v1:0603
- C9: value 10 uF -> 100nF; device rcl:C0805K -> freetronics-master-v1:0603
- D1, D10, D9: value UF4002 -> RS1D; device diode:D-7.5 -> freetronics-master-v1:SMA-DIODE
- D7: value 1N5819 -> RS1D; device diode:SOD123 -> freetronics-master-v1:SMA-DIODE
- D8: value 1N5819 -> SS16; device diode:SOD123 -> freetronics-luke:SMA
- IC11: value LMV7219M7 -> LMV7219M5
- IC14: value 74AHCT1G86GW -> SN74AHCT1G86DBVR
- IC3: value LD1117S50 -> APX811-44UG-7; device burr-brown:SOT223 -> freetronics-master-v1:SOT143-R
- J3: value Regulator Bypass -> CAN; device jumper:SJ -> con-molex:7395-04
- J5: value Terminator -> CAN Terminate; device jumper:SJ -> freetronics-luke:SJ
- J7: value CAN -> I2C; device con-subd:M09HP -> pinhead:1X02
- L2: value Bead -> 1uH; device inductor-neosid:SM-B5 -> rcl:L2012C
- LED1: value 60V -> 24V; device freetronics:LED-0805-LARGE -> freetronics-master-v1:LED-0603
- LED2: value 24V -> 5V; device freetronics:LED-0805-LARGE -> freetronics-master-v1:LED-0603
- LED3: value 5V -> Status; device freetronics:LED-0805-LARGE -> freetronics-master-v1:LED-0603
- LED5, LED6: device freetronics:LED-0805-LARGE -> freetronics-master-v1:LED-0603
- R10: value 13 k -> 260Ω; device rcl:M0805 -> rcl:R2010
- R11: value 1.5 k -> 10kΩ; device rcl:M0805 -> freetronics-master-v1:0603
- R13, R14: value 10 k -> 10kΩ; device rcl:M0805 -> freetronics-master-v1:0603
- R21: value 120 R -> 120Ω; device rcl:M0805 -> freetronics-master-v1:0603
- R23: value 130 k -> 3.9k; device resistor:M0805 -> freetronics-master-v1:0603
- R24: value 3.9 k -> 10kΩ; device resistor:M0805 -> freetronics-master-v1:0603
- R25: value 15 k -> 6.8k; device rcl:M0805 -> freetronics-master-v1:0603
- R26: value 6.8 k -> 1k; device rcl:M0805 -> freetronics-master-v1:0603
- R27, R38, R42: value 1 k -> 1k; device rcl:M0805 -> freetronics-master-v1:0603
- R30: value 10k -> 1kΩ; device resistor:M0805 -> freetronics-master-v1:0603
- R32: value 1 k -> 15k; device resistor:M0805 -> freetronics-master-v1:0603
- R46: value 10 k -> 130k; device rcl:M0805 -> freetronics-master-v1:0603
- R8, R9: value 0.43 R -> 10kΩ; device rcl:M0805 -> freetronics-master-v1:0603
- moved C29 96.6 mm to (1.27, 38.1), turned to 0 degrees
- moved R32 92.1 mm to (4.45, 43.2), turned to 180 degrees
- moved C28 86.6 mm to (1.27, 36.8), turned to 0 degrees
- moved C23 86.4 mm to (5.08, 36.8)
- moved R50 85.2 mm to (10.2, 35.6)
- moved R19 85.1 mm to (6.35, 39.4)
- moved C15 82.6 mm to (14.0, 38.1)
- moved C34 81.8 mm to (10.2, 35.6)
- moved R27 81.4 mm to (7.62, 30.5), turned to 0 degrees
- moved U$5 81.4 mm to (10.2, 36.8)
- moved C32 81.4 mm to (10.2, 35.6)
- moved R44 80.4 mm to (6.35, 34.3)
- moved C41 80.1 mm to (12.7, 43.2)
- moved R51 80.1 mm to (10.2, 40.6)
- moved C31 79.2 mm to (12.7, 33.0)
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Connections:
- removed net !THERM_CS: IC8.23
- removed net CAN_INT: IC8.4
- removed net N$26: D7.C, IC4.2, J3.1, L1.2
- removed net N$27: IC4.5, R10.1, R11.2
- removed net N$52: C16.1, J6.1
- removed net N$78: C15.2, IC8.34, Q5.2
- removed net N$79: C11.2, IC8.33, Q5.1
- removed net N$90: J7.5, J7.G1, J7.G2, J8.1
- removed net N$91: J5.1, R21.1
- removed net N$92: D8.C, J7.9
- removed net POT_1: C29.1, IC8.90, X1.2
- removed net POT_2: C28.1, IC8.91, X1.5
- removed net SCL: IC8.43
- removed net SDA: IC8.44
- new net N$19: IC20.26, J7.2
- new net N$24: C29.1, J6.1
- new net N$30: D8.A, J3.4
- new net N$31: J5.1, R21.2
- new net N$42: IC10.7, R66.1
- new net N$44: C55.1, IC10.3, L4.1
- new net N$51: C55.2, IC10.1
- new net N$59: C59.2, R62.2
- new net N$61: IC10.6, R62.1
- new net N$62: C54.2, IC10.8
- new net N$63: IC10.5, R63.2, R64.1
- new net N$65: C58.1, D18.A, L4.2, R63.1
- new net POT1: C16.1, IC20.55, X1.2
- new net POT2: C28.1, IC20.54, X1.5
- net !CAN_CS: now also IC20.10; no longer IC8.19
- net !CAN_INT: now also IC20.4
- net !RESET: now also IC20.20, IC3.2; no longer C16.2, IC8.30
- net +12V: now also C6.1, D7.A, ZD1.K; no longer C8.+, D2.A, IC3.3, L1.1
- net +24V: now also C57.1, D8.K, IC10.2, R10.1, R23.2, R25.1, R66.2; no longer C6.+, D8.A, IC4.6, J3.2, R24.2, R26.2, R8.1, R9.1
- net +5V: now also C12.2, C13.2, C15.1, C39.2, C43.2, C53.2, C7.2, D18.K, IC20.21, IC20.52, IC20.64, IC3.4, L2.2, R13.1, R26.1; no longer C14.2, C22.2, C37.1, C44.2, C45.2, C46.2, C9.1, IC3.2, IC8.10, IC8.100, IC8.31, IC8.61, IC8.80, L2.1, R27.2, R46.2
- net +5VA: now also C11.1, L2.1; no longer C21.2, L2.2
- net +60V: now also R32.1, R46.2; no longer R23.2, R25.2
- net 24V_MEASURE: now also C26.2, IC20.57, R23.1, R30.1; no longer C26.1, IC8.93, R24.1, R32.2
- net 60V_MEASURE: now also C25.2, IC20.56, R24.1, R46.1; no longer C25.1, IC8.92, R23.1, R30.2
- net AGND: now also C11.2, IC20.63; no longer C21.1, IC8.99
- net AREF: now also C8.2, IC20.62, R9.1; no longer C12.2, IC8.98, R13.1
- net BRIDGE_1_A: now also IC20.15; no longer IC8.24
- net BRIDGE_1_B: now also IC20.16; no longer IC8.25
- net BRIDGE_1_DIS: now also IC20.17; no longer IC8.26
- net BRIDGE_2_A: now also IC20.5; no longer IC8.5
- net BRIDGE_2_B: now also IC20.6; no longer IC8.6
- net BRIDGE_2_DIS: now also IC20.7; no longer IC8.7
- net CANH: now also J3.2, J5.2; no longer J7.7, R21.2
- net CANL: now also J3.1, R21.1; no longer J5.2, J7.2
- net CH1_CURRENT_SENSE: now also IC20.60; no longer IC8.96
- net CH1_GAIN_SELECT: now also IC20.61; no longer IC8.97
- net CH2_CURRENT_SENSE: now also IC20.58; no longer IC8.94
- net CH2_GAIN_SELECT: now also IC20.59; no longer IC8.95
- net D0: now also IC20.35; no longer IC8.53
- net D1: now also IC20.36; no longer IC8.54
- net D2: now also IC20.37; no longer IC8.55
- net D3: now also IC20.38; no longer IC8.56
- net D4: now also IC20.39; no longer IC8.57
- net D5: now also IC20.40; no longer IC8.58
- net D6: now also IC20.41; no longer IC8.59
- net D7: now also IC20.42; no longer IC8.60
- net DECODER_EN: now also IC20.30; no longer IC8.48
- net EN1: now also IC20.27; no longer IC8.45
- net EN2: now also IC20.28; no longer IC8.46
- net GND: now also C15.2, C16.2, C25.1, C26.1, C42.1, C43.1, C53.1, C54.1, C57.2, C58.2, C59.1, C6.2, C7.1, C8.1, C9.1, IC10.4, IC10.9, IC20.22, IC20.53, J3.3, LED7.C, R11.2, R24.2, R30.2, R64.2, R8.2, ZD1.A; no longer C11.1, C15.1, C22.1, C25.2, C26.2, C29.2, C36.1, C37.2, C44.1, C45.1, C46.1, C6.-, C7.2, C8.-, C9.2, D7.A, IC4.4, IC8.11, IC8.32, IC8.62, IC8.81, J7.3, J7.6, J8.2, LED4.C, R11.1, R14.1, R30.1, R32.1, R53.1
- net LED: now also IC20.14, R27.1; no longer IC8.8, R28.2
- net MAIN_CLK: now also IC20.24, R14.1; no longer R49.1
- net MISO: now also IC20.13; no longer IC8.22
- net MOSI: now also IC20.12; no longer IC8.21
- net N$10: now also J11.1; no longer J11.2
- net N$12: now also J11.2; no longer J11.1
- net N$13: now also LED2.A, R26.2; no longer LED3.A, R27.1
- net N$14: now also C9.2, R8.1, R9.2; no longer C13.2, R13.2, R14.2
- net N$20: now also IC20.25, J7.1; no longer IC4.1, IC4.7, IC4.8, R8.2, R9.2
- net N$23: now also C29.2, IC3.3; no longer C7.1, IC4.3
- net N$3: now also C14.2, R14.2; no longer C36.2, R49.2
- net N$43: now also LED1.A, R25.2; no longer LED2.A, R26.1
- net N$5: now also R11.1, R13.2; no longer R46.1, R53.2
- net N$50: now also LED3.A, R27.2; no longer LED4.A, R28.1
- net N$55: now also LED7.A, R32.2; no longer LED1.A, R25.1
- net N$56: now also C38.2; no longer C39.2
- net N$57: now also C42.2; no longer C38.2
- net N$60: now also D10.C; no longer D1.C
- net N$66: now also D1.C; no longer D2.C
- net N$89: now also D7.C; no longer D9.C
- net N$93: now also D9.C; no longer D10.C
- net RSTX: now also IC20.32; no longer IC8.50
- net RSTY: now also IC20.31; no longer IC8.49
- net RXD: now also IC20.2; no longer IC8.2
- net SCK: now also IC20.11; no longer IC8.20
- net SEL1: now also IC20.29; no longer IC8.47
- net SEL2: now also IC20.33; no longer IC8.51
- net TXD: now also IC20.3; no longer IC8.3
- net X/Y: now also IC20.34; no longer IC8.52
Routing:
- net N$82: track 0.00 -> 53.2 mm, vias 0 -> 2
- net +5V: track 47.1 -> 0.00 mm, vias 4 -> 0
- net N$74: track 11.4 -> 55.9 mm, vias 0 -> 3
- net N$88: track 0.00 -> 37.5 mm, vias 0 -> 1
- net N$80: track 10.8 -> 47.3 mm, vias 0 -> 1
- net N$81: track 0.00 -> 36.0 mm
- net N$8: track 31.8 -> 0.00 mm
- net N$12: track 30.1 -> 0.00 mm
- net N$7: track 29.3 -> 0.00 mm
- net N$10: track 28.7 -> 0.00 mm
- net N$9: track 24.8 -> 0.00 mm
- net D3: track 24.2 -> 0.00 mm, vias 1 -> 0
- net D2: track 24.2 -> 0.00 mm, vias 1 -> 0
- net D1: track 24.2 -> 0.00 mm, vias 1 -> 0
- net N$1: track 23.6 -> 0.00 mm
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