File: OpenServoDrive.sch (EAGLE design)
At the start: 175 parts, among them IC1 LTC6103, IC11 LMV7219M7, IC12 MCP2515, IC13 HCTL-2032-SC, IC14 74AHCT1G86GW, IC15 MCP2551, IC16 HIP4081A, IC2 HIP4081A, IC3 LD1117S50, IC4 MC34063, IC5 OPA336NJ, IC6 OPA2336UA, IC7 OPA2336UA, IC8 ATMEGA2560-16AU, IC9 LTC6103, J1 Motor 1, J13 Motor 2, J2 60V Motor Power, J3 Regulator Bypass, J4 AREF, J5 Terminator, J7 CAN, J8 Ground, J9 ISP, Q1 AOT414, Q10 AOT414, Q11 16 MHz, Q12 2N7002, Q13 16 MHz, Q2 AOT414, Q3 AOT414, Q4 AOT414, Q5 16 MHz, Q6 2N7002, Q7 AOT414, Q8 AOT414, Q9 AOT414

Commit message: foo
Parts:
- removed C21, C22, C44, C45, C46: 100 nF, rcl:C-EUC0805K
- removed C36: 22 pF, rcl:C-EUC0805K
- removed C37: 100nF, rcl:C-EUC0805K
- removed D2: UF4002, diode:DIODE-D-7.5
- removed IC4: MC34063, SparkFun:MC34063SMD
- removed IC8: ATMEGA2560-16AU, atmel-2005:ATMEGA1280-16AU
- removed J8: Ground, jumper:SJ
- removed L1: 220 uH, wuerth-elektronik:WE-PD_L/XL/XXL
- removed LED4: Status, freetronics:LED0805-LARGE
- removed Q5: 16 MHz, SparkFun:CRYSTALHC49US
- removed R28, R49: 1 k, rcl:R-US_M0805
- removed R53: 10 k, rcl:R-US_M0805
- removed U$3, U$6, U$7: OSHW-LOGOS, SparkFun:OSHW-LOGOS
- added C42: 22pF, freetronics-master-v1:CAP0603
- added C43, C54: 100nF, freetronics-master-v1:CAP0603
- added C53, C59: 2.2nF, freetronics-master-v1:CAP0603
- added C55: 10nF, freetronics-master-v1:CAP0603
- added C57: 10µF, freetronics-jon:C-EUC1206K
- added C58: 22µF, freetronics-jon:C-EUC1206K
- added D18: SK34A-LTP, freetronics-luke:SCHOTTKY
- added IC10: EUP3476, freetronics-luke:EUP3476
- added IC20: ATmega1281, SparkFun:ATMEGA128-SMD
- added L4: 6.8 uH, freetronics-luke:INDUCTOR
- added LED7: 60V, freetronics-master-v1:LED0603
- added R62: 15k, freetronics-master-v1:RESISTOR0603
- added R63: 53.6k, freetronics-master-v1:RESISTOR0603
- added R64: 10k 1%, freetronics-master-v1:RESISTOR0603
- added R66: 100k, freetronics-master-v1:RESISTOR0603
- added U$55, U$56, U$68: OSHW-LOGOS, SparkFun:OSHW-LOGOS
- added ZD1: 12.6V, freetronics-luke:ZENERMINIMELF
- C11, C15, C39: value 22 pF -> 100nF; device rcl:C-EUC0805K -> freetronics-master-v1:CAP0603; PACKAGE (none) -> 0603
- C12, C13: value 100 nF -> 100nF; device rcl:C-EUC0805K -> freetronics-master-v1:CAP0603; PACKAGE (none) -> 0603
- C14: value 100 nF -> 22pF; device rcl:C-EUC0805K -> freetronics-master-v1:CAP0603; PACKAGE (none) -> 0603
- C16: value 100 nF -> 10nF; device rcl:C-EUC0805K -> freetronics-master-v1:CAP0603; PACKAGE (none) -> 0603
- C25, C26, C28: value 10 nF -> 10nF; device rcl:C-EUC0805K -> freetronics-master-v1:CAP0603; PACKAGE (none) -> 0603
- C29: value 10 nF -> 100nF; device rcl:C-EUC0805K -> freetronics-master-v1:CAP0603; PACKAGE (none) -> 0603
- C38: value 22 pF -> 22pF; device rcl:C-EUC0805K -> freetronics-master-v1:CAP0603; PACKAGE (none) -> 0603
- C6: value 100 uF -> 47µF; device resistor:CPOL-EUE2.5-6 -> freetronics-jon:C-EUC1210; VOLTAGE (none) -> 16V 1210
- C7: value 470 pF -> 100nF; device rcl:C-EUC0805K -> freetronics-master-v1:CAP0603; PACKAGE (none) -> 0603
- C8: value 470 uF -> 100nF; device resistor:CPOL-EUE3.5-8 -> freetronics-master-v1:CAP0603; PACKAGE (none) -> 0603
- C9: value 10 uF -> 100nF; device rcl:C-EUC0805K -> freetronics-master-v1:CAP0603; PACKAGE (none) -> 0603
- D1, D10, D9: value UF4002 -> RS1D; device diode:DIODE-D-7.5 -> freetronics-master-v1:DIODESMA; PACKAGE (none) -> SMA
- D7: value 1N5819 -> RS1D; device diode:DIODE-SOD123 -> freetronics-master-v1:DIODESMA; PACKAGE (none) -> SMA
- D8: value 1N5819 -> SS16; device diode:DIODE-SOD123 -> freetronics-luke:SCHOTTKY; PACKAGE (none) -> SMA
- IC11: value LMV7219M7 -> LMV7219M5; PACKAGE (none) -> SOT23-5
- IC14: value 74AHCT1G86GW -> SN74AHCT1G86DBVR; PACKAGE (none) -> SOT23-5
- IC3: value LD1117S50 -> APX811-44UG-7; device burr-brown:REG1117 -> freetronics-master-v1:APX81X-RESET-IC
- IC5: PACKAGE (none) -> SOT23-5
- J3: value Regulator Bypass -> CAN; device jumper:SJ -> con-molex:22-05-7048-04
- J5: value Terminator -> CAN Terminate; device jumper:SJ -> freetronics-luke:SJ
- J7: value CAN -> I2C; device con-subd:M09HP -> pinhead:PINHD-1X2
- L2: value Bead -> 1uH; device inductor-neosid:SM-B5 -> rcl:L-USL2012C; CURRENT (none) -> 250mA; PACKAGE (none) -> 0805
- LED1: value 60V -> 24V; device freetronics:LED0805-LARGE -> freetronics-master-v1:LED0603
- LED2: value 24V -> 5V; device freetronics:LED0805-LARGE -> freetronics-master-v1:LED0603
- LED3: value 5V -> Status; device freetronics:LED0805-LARGE -> freetronics-master-v1:LED0603
- LED5, LED6: device freetronics:LED0805-LARGE -> freetronics-master-v1:LED0603
- Q13: SKU (none) -> CTX270CT-ND
- R10: value 13 k -> 260Ω; device rcl:R-US_M0805 -> rcl:R-EU_R2010; PACKAGE (none) -> 1W 2010
- R11: value 1.5 k -> 10kΩ; device rcl:R-US_M0805 -> freetronics-master-v1:RESISTOR0603; PACKAGE (none) -> 0603
- R13, R14: value 10 k -> 10kΩ; device rcl:R-US_M0805 -> freetronics-master-v1:RESISTOR0603; PACKAGE (none) -> 0603
- R21: value 120 R -> 120Ω; device rcl:R-US_M0805 -> freetronics-master-v1:RESISTOR0603; PACKAGE (none) -> 0603
- R23: value 130 k -> 3.9k; device resistor:R-US_M0805 -> freetronics-master-v1:RESISTOR0603; PACKAGE (none) -> 0603
- R24: value 3.9 k -> 10kΩ; device resistor:R-US_M0805 -> freetronics-master-v1:RESISTOR0603; PACKAGE (none) -> 0603
- R25: value 15 k -> 6.8k; device rcl:R-US_M0805 -> freetronics-master-v1:RESISTOR0603; PACKAGE (none) -> 0603
- R26: value 6.8 k -> 1k; device rcl:R-US_M0805 -> freetronics-master-v1:RESISTOR0603; PACKAGE (none) -> 0603
- R27, R38, R42: value 1 k -> 1k; device rcl:R-US_M0805 -> freetronics-master-v1:RESISTOR0603; PACKAGE (none) -> 0603
- R30: value 10k -> 1kΩ; device resistor:R-US_M0805 -> freetronics-master-v1:RESISTOR0603; PACKAGE (none) -> 0603
- R32: value 1 k -> 15k; device resistor:R-US_M0805 -> freetronics-master-v1:RESISTOR0603; PACKAGE (none) -> 0603
- R46: value 10 k -> 130k; device rcl:R-US_M0805 -> freetronics-master-v1:RESISTOR0603; PACKAGE (none) -> 0603
- R8, R9: value 0.43 R -> 10kΩ; device rcl:R-US_M0805 -> freetronics-master-v1:RESISTOR0603; PACKAGE (none) -> 0603
Connections:
- removed net !THERM_CS: IC8.(OC2A/PCINT4)PB4
- removed net CAN_INT: IC8.(XCK0/AIN0)PE2
- removed net N$26: D7.C, IC4.SWE, J3.1, L1.1
- removed net N$27: IC4.COMP, R10.1, R11.2
- removed net N$52: C16.1, J6.DTR
- removed net N$78: C15.2, IC8.XTAL1, Q5.2
- removed net N$79: C11.2, IC8.XTAL2, Q5.1
- removed net N$90: J7.5, J7.G1, J7.G2, J8.1
- removed net N$91: J5.1, R21.1
- removed net N$92: D8.C, J7.9
- removed net POT_1: C29.1, IC8.(ADC7/TDI)PF7, X1-2.1
- removed net POT_2: C28.1, IC8.(ADC6/TDO)PF6, X1-5.1
- removed net SCL: IC8.(SCL/INT0)PD0
- removed net SDA: IC8.(SDA/INT1)PD1
- new net N$19: IC20.PD1(SDA), J7.2
- new net N$24: C29.1, J6.DTR
- new net N$30: D8.A, J3-4.S
- new net N$31: J5.1, R21.2
- new net N$42: IC10.EN, R66.1
- new net N$44: C55.1, IC10.SW, L4.1
- new net N$51: C55.2, IC10.BS
- new net N$59: C59.2, R62.2
- new net N$61: IC10.COMP, R62.1
- new net N$62: C54.2, IC10.SS
- new net N$63: IC10.FB, R63.2, R64.1
- new net N$65: C58.1, D18.A, L4.2, R63.1
- new net POT1: C16.1, IC20.PF6, X1-2.1
- new net POT2: C28.1, IC20.PF7, X1-5.1
- net !CAN_CS: now also IC20.PB0(SS); no longer IC8.(SS/PCINT0)PB0
- net !CAN_INT: now also IC20.PE2
- net !RESET: now also IC20.RESET, IC3./RESET; no longer C16.2, IC8.RESET
- net +12V: now also C6.1, D7.A, ZD1.K; no longer C8.+, D2.A, IC3.VIN, L1.2
- net +24V: now also C57.1, D8.K, IC10.IN, R10.1, R23.2, R25.1, R66.2; no longer C6.+, D8.A, IC4.VCC, J3.2, R24.2, R26.2, R8.1, R9.1
- net +5V: now also C12.2, C13.2, C15.1, C39.2, C43.2, C53.2, C7.2, D18.K, IC20.AVCC, IC20.VCC@21, IC20.VCC@52, IC3.VCC, L2.2, R13.1, R26.1; no longer C14.2, C22.2, C37.1, C44.2, C45.2, C46.2, C9.1, IC3.VOUT, IC8.AVCC, IC8.VCC, IC8.VCC1, IC8.VCC2, IC8.VCC3, L2.1, R27.2, R46.2
- net +5VA: now also C11.1, L2.1; no longer C21.2, L2.2
- net +60V: now also R32.1, R46.2; no longer R23.2, R25.2
- net 24V_MEASURE: now also C26.2, IC20.PF4, R23.1, R30.1; no longer C26.1, IC8.(ADC4/TCK)PF4, R24.1, R32.2
- net 60V_MEASURE: now also C25.2, IC20.PF5, R24.1, R46.1; no longer C25.1, IC8.(ADC5/TMS)PF5, R23.1, R30.2
- net AGND: now also C11.2, IC20.AGND; no longer C21.1, IC8.AGND
- net AREF: now also C8.2, IC20.AREF, R9.1; no longer C12.2, IC8.AREF, R13.1
- net BRIDGE_1_A: now also IC20.PB5; no longer IC8.(OC1A/PCINT5)PB5
- net BRIDGE_1_B: now also IC20.PB6; no longer IC8.(OC1B/PCINT6)PB6
- net BRIDGE_1_DIS: now also IC20.PB7; no longer IC8.(OC0A/OC1C/PCINT7)PB7
- net BRIDGE_2_A: now also IC20.PE3; no longer IC8.(OC3A/AIN1)PE3
- net BRIDGE_2_B: now also IC20.PE4; no longer IC8.(OC3B/INT4)PE4
- net BRIDGE_2_DIS: now also IC20.PE5; no longer IC8.(OC3C/INT5)PE5
- net CANH: now also J3-2.S, J5.2; no longer J7.7, R21.2
- net CANL: now also J3-1.S, R21.1; no longer J5.2, J7.2
- net CH1_CURRENT_SENSE: now also IC20.PF1; no longer IC8.(ADC1)PF1
- net CH1_GAIN_SELECT: now also IC20.PF0; no longer IC8.(ADC0)PF0
- net CH2_CURRENT_SENSE: now also IC20.PF3; no longer IC8.(ADC3)PF3
- net CH2_GAIN_SELECT: now also IC20.PF2; no longer IC8.(ADC2)PF2
- net D0: now also IC20.PC0; no longer IC8.(A8)PC0
- net D1: now also IC20.PC1; no longer IC8.(A9)PC1
- net D2: now also IC20.PC2; no longer IC8.(A10)PC2
- net D3: now also IC20.PC3; no longer IC8.(A11)PC3
- net D4: now also IC20.PC4; no longer IC8.(A12)PC4
- net D5: now also IC20.PC5; no longer IC8.(A13)PC5
- net D6: now also IC20.PC6; no longer IC8.(A14)PC6
- net D7: now also IC20.PC7; no longer IC8.(A15)PC7
- net DECODER_EN: now also IC20.PD5; no longer IC8.(XCK1)PD5
- net EN1: now also IC20.PD2; no longer IC8.(RXD1/INT2)PD2
- net EN2: now also IC20.PD3; no longer IC8.(TXD1/INT3)PD3
- net GND: now also C15.2, C16.2, C25.1, C26.1, C42.1, C43.1, C53.1, C54.1, C57.2, C58.2, C59.1, C6.2, C7.1, C8.1, C9.1, IC10.GND, IC10.TGND, IC20.GND@22, IC20.GND@53, J3-3.S, LED7.C, R11.2, R24.2, R30.2, R64.2, R8.2, ZD1.A; no longer C11.1, C15.1, C22.1, C25.2, C26.2, C29.2, C36.1, C37.2, C44.1, C45.1, C46.1, C6.-, C7.2, C8.-, C9.2, D7.A, IC4.GND, IC8.GND, IC8.GND1, IC8.GND2, IC8.GND3, J7.3, J7.6, J8.2, LED4.C, R11.1, R14.1, R30.1, R32.1, R53.1
- net LED: now also IC20.PB4, R27.1; no longer IC8.(T3/INT6)PE6, R28.2
- net MAIN_CLK: now also IC20.XTAL1, R14.1; no longer R49.1
- net MISO: now also IC20.PB3(MISO); no longer IC8.(MISO/PCINT3)PB3
- net MOSI: now also IC20.PB2(MOSI); no longer IC8.(MOSI/PCINT2)PB2
- net N$10: now also J11.1; no longer J11.2
- net N$12: now also J11.2; no longer J11.1
- net N$13: now also LED2.A, R26.2; no longer LED3.A, R27.1
- net N$14: now also C9.2, R8.1, R9.2; no longer C13.2, R13.2, R14.2
- net N$20: now also IC20.PD0(SCL), J7.1; no longer IC4.DVR, IC4.SEN, IC4.SWC, R8.2, R9.2
- net N$23: now also C29.2, IC3./MR; no longer C7.1, IC4.TC
- net N$3: now also C14.2, R14.2; no longer C36.2, R49.2
- net N$43: now also LED1.A, R25.2; no longer LED2.A, R26.1
- net N$5: now also R11.1, R13.2; no longer R46.1, R53.2
- net N$50: now also LED3.A, R27.2; no longer LED4.A, R28.1
- net N$55: now also LED7.A, R32.2; no longer LED1.A, R25.1
- net N$56: now also C38.2; no longer C39.2
- net N$57: now also C42.2; no longer C38.2
- net N$60: now also D10.C; no longer D1.C
- net N$66: now also D1.C; no longer D2.C
- net N$89: now also D7.C; no longer D9.C
- net N$93: now also D9.C; no longer D10.C
- net RSTX: now also IC20.PD7; no longer IC8.(T0)PD7
- net RSTY: now also IC20.PD6; no longer IC8.(T1)PD6
- net RXD: now also IC20.PE0(RXD); no longer IC8.(RXD0/PCIN8)PE0
- net SCK: now also IC20.PB1(SCK); no longer IC8.(SCK/PCINT1)PB1
- net SEL1: now also IC20.PD4; no longer IC8.(ICP1)PD4
- net SEL2: now also IC20.PG0; no longer IC8.(WR)PG0
- net TXD: now also IC20.PE1(TXD); no longer IC8.(TXD0)PE1
- net X/Y: now also IC20.PG1; no longer IC8.(RD)PG1
Other:
- note added: "28-SOIC Wide"
- note added: "AVR ADC's differential input is limited to 4 kHz bandwidth so a single-ended output is needed."
- note added: "CAN connector and power supplies"
- note added: "HCTL-2032-SC"
- note added: "If input voltage is 12V already, 260Ω resistor can be shorted and the Zener omitted."
- note removed: "(one end only to prevent ground loop)"
- note removed: "0.43R, 0.25W, 1%, 0805"
- note removed: "12 volts, remove the IC and short the jumper."
- note removed: "16 MHz oscillator"
- note removed: "16V"
- note removed: "2 x"
- note removed: "35V"
- note removed: "399-6104-ND"
- note removed: "732-1688-1-ND"
- note removed: "AVR ADC's differential input is limited to 4 kHz bandwidth"
- note removed: "Avago HCTL-2032-SC"
- note removed: "C8: 493-1043-ND"
- note removed: "C9: 445-1371-1-ND"
- note removed: "CAN connector (DE-9)"
- note removed: "CTX270CT-ND"
- note removed: "D7: 1N5819HW-FDICT-ND"
- note removed: "If the 12V input feed is already regulated"
- note removed: "Input voltage probably 24V, may be 12V-30V."
- note removed: "J5: CAN bus terminator on/off"
- note removed: "J8: CAN bus shield to ground"
- note removed: "Microcontroller (ATmega2560)"
- note removed: "Motor 1 current feedback amplifier"
- note removed: "Motor 2 current feedback amplifier"
- note removed: "RHM.43MCT-ND"
- note removed: "Ref. = 1.25 V"
- note removed: "Voltage Regulators"
- note removed: "so a single-ended output is needed."
- moved on the sheet: C1, C10, C11, C12, C13, C14, C15, C16, C17, C18, C19, C2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
